File: HW/STM32-FC/memory.kicad_sch (KiCad schematic)
At the start: 9 parts, among them J4 TF-06A, U6 W25X40CLUXIG

Commit message: HW Lib and RC code refactoring, GCS_log united and BMI323 IMU init.
Parts:
- J4: footprint TF-06A:TF06A -> TF06A
Changed lines of the file:
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@@
 	(title_block
 		(title "Memory")
-		(date "2025-04-13")
+		(date "2025-06-19")
 		(rev "A")
 		(company "NARAE")
@@
 			)
 		)
-		(property "Footprint" "TF-06A:TF06A"
+		(property "Footprint" "TF06A"
 			(at 177.8 127.94 0)
 			(effects
